File: staggered-keyboard.kicad_pcb (KiCad board)
At the start: 2 copper layers, 306.4 x 95.3 mm, 129 parts, among them U1 ProMicro

Commit message: Fix errors after running DRC
Routing:
- net Row 2: track 320.0 -> 301.6 mm
- net Row 3: track 339.5 -> 324.3 mm
- net Row 1: track 295.9 -> 281.4 mm
- net Row 4: track 436.4 -> 423.2 mm
Other:
- board size 306.4 x 95.3 mm -> 306.4 x 96.4 mm
Changed lines of the file:
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@@
     )
   )
-  (gr_arc (start 67.46875 234.95) (mid 65.784952 234.252548) (end 65.0875 232.56875) (layer "Edge.Cuts") (width 0.1))
-  (gr_line (start 67.46875 234.95) (end 369.09375 234.95) (layer "Edge.Cuts") (width 0.1))
-  (gr_arc (start 368.264936 139.660064) (mid 370.51 140.59) (end 371.439936 142.835064) (layer "Edge.Cuts") (width 0.1))
-  (gr_arc (start 371.475 232.56875) (mid 370.777548 234.252548) (end 369.09375 234.95) (layer "Edge.Cuts") (width 0.1))
-  (gr_line (start 65.102548 142.083798) (end 65.102548 232.571298) (layer "Edge.Cuts") (width 0.1))
-  (gr_line (start 371.475 232.56875) (end 371.439936 142.87) (layer "Edge.Cuts") (width 0.1))
-  (gr_line (start 368.3 139.7) (end 67.483798 139.702548) (layer "Edge.Cuts") (width 0.1))
+  (gr_arc (start 67.493798 236.077452) (mid 65.810015 235.379985) (end 65.112548 233.696202) (layer "Edge.Cuts") (width 0.1))
+  (gr_line (start 67.493798 236.077452) (end 369.11875 236.08125) (layer "Edge.Cuts") (width 0.1))
+  (gr_arc (start 368.264947 139.67) (mid 370.51 140.599947) (end 371.439947 142.845) (layer "Edge.Cuts") (width 0.1))
+  (gr_arc (start 371.5 233.7) (mid 370.802533 235.383783) (end 369.11875 236.08125) (layer "Edge.Cuts") (width 0.1))
+  (gr_line (start 65.102548 142.083798) (end 65.112548 233.696202) (layer "Edge.Cuts") (width 0.1))
+  (gr_line (start 371.5 233.7) (end 371.439947 142.845) (layer "Edge.Cuts") (width 0.1))
+  (gr_line (start 368.264947 139.67) (end 67.483798 139.702548) (layer "Edge.Cuts") (width 0.1))
   (gr_arc (start 65.102548 142.083798) (mid 65.8 140.4) (end 67.483798 139.702548) (layer "Edge.Cuts") (width 0.1))
   (segment (start 141.46 153.45) (end 331.9 153.45) (width 0.25) (layer "B.Cu") (net 1))
@@
   (segment (start 79.6255 172.55) (end 108.21 172.55) (width 0.25) (layer "B.Cu") (net 16))
   (segment (start 341.38 172.67) (end 108.33 172.67) (width 0.25) (layer "B.Cu") (net 16))
-  (segment (start 93.75 172.55) (end 108.21 172.55) (width 0.25) (layer "B.Cu") (net 16))
   (segment (start 341.53 172.52) (end 341.38 172.67) (width 0.25) (layer "B.Cu") (net 16))
   (segment (start 108.33 172.67) (end 108.21 172.55) (width 0.25) (layer "B.Cu") (net 16))
@@
   (segment (start 80.35 160.13) (end 83.3 157.18) (width 0.25) (layer "F.Cu") (net 31))
   (segment (start 80.3555 191.6) (end 80.35 191.5945) (width 0.25) (layer "F.Cu") (net 31))
-  (segment (start 83.3 157.18) (end 83.3 157.52) (width 0.25) (layer "F.Cu") (net 31))
   (via (at 80.3555 191.6) (size 0.8) (drill 0.4) (layers "F.Cu" "B.Cu") (net 31))
-  (segment (start 92.54 191.6) (end 110.65 191.6) (width 0.25) (layer "B.Cu") (net 31))
+  (segment (start 80.3555 191.6) (end 110.65 191.6) (width 0.25) (layer "B.Cu") (net 31))
   (segment (start 110.65 191.6) (end 346.25 191.6) (width 0.25) (layer "B.Cu") (net 31))
   (segment (start 346.25 191.6) (end 346.28 191.57) (width 0.25) (layer "B.Cu") (net 31))
-  (segment (start 80.3555 191.6) (end 110.65 191.6) (width 0.25) (layer "B.Cu") (net 31))
   (segment (start 104.93375 182.245) (end 110.65 187.96125) (width 0.25) (layer "B.Cu") (net 32))
   (segment (start 110.65 187.96125) (end 110.65 188.3) (width 0.25) (layer "B.Cu") (net 32))
@@
   (segment (start 346.28 187.8775) (end 346.28 188.27) (width 0.25) (layer "B.Cu") (net 44))
   (segment (start 340.63 182.2275) (end 346.28 187.8775) (width 0.25) (layer "B.Cu") (net 44))
-  (segment (start 81.09 161.93) (end 81.09 210.5655) (width 0.25) (layer "F.Cu") (net 45))
-  (segment (start 81.0755 210.58) (end 81.0755 210.4345) (width 0.25) (layer "F.Cu") (net 45))
-  (segment (start 81.09 210.5655) (end 81.0755 210.58) (width 0.25) (layer "F.Cu") (net 45))
-  (segment (start 81.09 161.93) (end 83.3 159.72) (width 0.25) (layer "F.Cu") (net 45))
-  (segment (start 83.3 159.72) (end 83.3 159.79) (width 0.25) (layer "F.Cu") (net 45))
-  (via (at 81.0755 210.58) (size 0.8) (drill 0.4) (layers "F.Cu" "B.Cu") (net 45))
+  (segment (start 81.07 191.289195) (end 81.07 161.95) (width 0.25) (layer "F.Cu") (net 45))
+  (segment (start 81.0805 191.299695) (end 81.07 191.289195) (width 0.25) (layer "F.Cu") (net 45))
+  (segment (start 81.0805 191.900305) (end 81.0805 191.299695) (width 0.25) (layer "F.Cu") (net 45))
+  (segment (start 81.07 191.910805) (end 81.0805 191.900305) (width 0.25) (layer "F.Cu") (net 45))
+  (segment (start 81.07 210.56) (end 81.07 191.910805) (width 0.25) (layer "F.Cu") (net 45))
+  (segment (start 81.07 161.95) (end 83.3 159.72) (width 0.25) (layer "F.Cu") (net 45))
+  (via (at 81.07 210.57) (size 0.8) (drill 0.4) (layers "F.Cu" "B.Cu") (net 45))
   (segment (start 353.52 210.58) (end 353.56 210.54) (width 0.25) (layer "B.Cu") (net 45))
-  (segment (start 81.0755 210.58) (end 105.8 210.58) (width 0.25) (layer "B.Cu") (net 45))
-  (segment (start 91 210.58) (end 105.8 210.58) (width 0.25) (layer "B.Cu") (net 45))
+  (segment (start 81.07 210.57) (end 81.08 210.58) (width 0.25) (layer "B.Cu") (net 45))
+  (segment (start 81.08 210.58) (end 105.8 210.58) (width 0.25) (layer "B.Cu") (net 45))
   (segment (start 105.8 210.58) (end 353.52 210.58) (width 0.25) (layer "B.Cu") (net 45))
-  (segment (start 83.12 159.72) (end 83.3 159.72) (width 0.25) (layer "B.Cu") (net 45))
   (segment (start 100.17125 201.295) (end 105.8 206.92375) (width 0.25) (layer "B.Cu") (net 46))
   (segment (start 105.8 206.92375) (end 105.8 207.28) (width 0.25) (layer "B.Cu") (net 46))
@@
   (segment (start 81.88 229.73) (end 103.48 229.73) (width 0.25) (layer "B.Cu") (net 59))
   (segment (start 360.65 218.36) (end 361.18 217.83) (width 0.25) (layer "B.Cu") (net 59))
-  (segment (start 90.43 229.73) (end 103.48 229.73) (width 0.25) (layer "B.Cu") (net 59))
   (segment (start 361.18 215.58) (end 361.18 189.56) (width 0.25) (layer "B.Cu") (net 59))
   (segment (start 361.18 189.56) (end 366.67 184.07) (width 0.25) (layer "B.Cu") (net 59))
-  (segment (start 83.12 162.26) (end 83.3 162.26) (width 0.25) (layer "B.Cu") (net 59))
   (segment (start 355.07 157.57) (end 355.07 159.14) (width 0.25) (layer "B.Cu") (net 59))
   (segment (start 351.37 229.7) (end 354.75 226.32) (width 0.25) (layer "B.Cu") (net 59))

Commit message: Update pcb design && various changes
- Generate Gerber file for production
- Generate .step file for 3D design
Parts:
- added ?: , , F.Cu at (349.4, 219.1)
- added ?: , , F.Cu at (228.6, 219.1)
- added ?: , , F.Cu at (222.1, 158.9)
- added ?: , , F.Cu at (87.2, 218.9)
- added ?: , , F.Cu at (87.0, 157.5)
- added REF**: MountingHole_3.2mm_M3, MountingHole:MountingHole_3.2mm_M3, F.Cu at (349.8, 158.8)
Other:
- board size 306.4 x 96.4 mm -> 306.5 x 97 mm
- board text added: "<- M3"
- board text added: "@PeuTit"

Commit message: Add hotswap socket to pcb
Parts:
- removed ? (x5): , 
- removed REF**: MountingHole_3.2mm_M3, MountingHole:MountingHole_3.2mm_M3
- MX1, MX10, MX11, MX12, MX13, MX16, MX17, MX18, MX19, MX2, MX20, MX21, MX22, MX23, MX24, MX25, MX26, MX27, MX3, MX30, MX31, MX32, MX33, MX34, MX35, MX36, MX37, MX38, MX39, MX4, MX40, MX41, MX43, MX44, MX45, MX46, MX47, MX48, MX49, MX5, MX50, MX51, MX52, MX53, MX55, MX6, MX64, MX7, MX8, MX9: footprint MX_Only:MXOnly-1U-NoLED -> MX_Only:MXOnly-1U-Hotswap
- MX14: footprint MX_Only:MXOnly-2U-NoLED -> MX_Only:MXOnly-2U-Hotswap
- MX15: footprint MX_Only:MXOnly-1.5U-NoLED -> MX_Only:MXOnly-1.5U-Hotswap
- MX28: footprint MX_Only:MXOnly-ISO-NoLED -> MX_Only:MXOnly-ISO-Hotswap-ReversedStabilizers
- MX29: footprint MX_Only:MXOnly-1.75U-NoLED -> MX_Only:MXOnly-1.75U-Hotswap
- MX42, MX56, MX57, MX58, MX61, MX62, MX63: footprint MX_Only:MXOnly-1.25U-NoLED -> MX_Only:MXOnly-1.25U-Hotswap
- MX54: footprint MX_Only:MXOnly-2.75U-NoLED -> MX_Only:MXOnly-2.75U-Hotswap
- MX59, MX60: footprint MX_Only:MXOnly-2.75U-NoLED -> MX_Only:MXOnly-2.75U-Hotswap-ReversedStabilizers
- moved D14 6.99 mm to (360.6, 151.7)
- moved D28 0.51 mm to (363.4, 169.0)
Routing:
- net Col 8: track 283.3 -> 306.4 mm, vias 2 -> 7
- net Col 2: track 140.4 -> 155.5 mm, vias 1 -> 6
- net Col 5: track 238.6 -> 253.1 mm, vias 2 -> 7
- net Col 3: track 171.9 -> 184.3 mm, vias 0 -> 5
- net Col 6: track 401.0 -> 413.1 mm, vias 3 -> 7
- net Col 1: track 120.5 -> 132.1 mm, vias 1 -> 6
- net Col 4: track 174.5 -> 182.8 mm, vias 0 -> 4
- net Col 0: track 94.1 -> 99.7 mm, vias 1 -> 6
- net Col 10: track 352.2 -> 357.2 mm, vias 2 -> 7
- net Col 11: track 372.9 -> 377.3 mm, vias 2 -> 7
- net Row 4: track 423.2 -> 426.8 mm
- net Net-(D14-Pad2): track 10.2 -> 6.86 mm
- net Col 9: track 409.2 -> 407.1 mm, vias 4 -> 7
- net Col 7: track 379.1 -> 381.2 mm, vias 2 -> 6
- net Net-(D28-Pad2): track 3.32 -> 5.22 mm
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Other:
- board size 306.5 x 97 mm -> 307 x 96 mm
- board text removed: "<- M3"
